File: hardware/mollusk-pedal.sch (KiCad schematic (older format))
At the start: 30 parts

Commit message: Fixed up input signal path.
Parts:
- removed R?: R, symbol R
- added R?: 22k, symbol R
- added R? (x3): 1k, symbol R
- added R?: 5.1k, symbol R
- C? (x2): value C -> 10uF
- C?: value C -> 5.1k
- C?: value C -> .01uF
- R? (x2): value R -> 2M
- R?: value R -> .01uF
- R? (x3): value R -> 360
Connections:
- net GND: now also C?.1, R?.1
- net MOSI: now also R?.1
- net VCC: now also R?.1
- net at C?.2, U?.5 (+): now also R?.2
- net at C?.1, U?.1: now also R?.2; no longer U?.2 (-)
- net at IC?.6 ((PCINT7/ICP/OC0B/ADC7)PA7): no longer C?.1
- new net: R?.1, R?.1, U?.2 (-)
- new net: R?.2, R?.2, R?.2
- no-connect marks 0 -> 1
Other:
- moved on the sheet: C?, CON?, R?
